File: PanTermPCB/PanTermPCB.kicad_sch (KiCad schematic)
At the start: 0 parts

Commit message: Basic esp32 wroom1 circuitry
Parts:
- added C11, C8: CL10A106KP8NNNC 10uF, lcsc_footprints:C19702_C0603, symbol lcsc_imported:CL10A106KP8NNNC
- added C7: 100nF (104) ±10% 50V, lcsc_footprints:C1591_C0603, symbol lcsc_imported:100nF_(104)_±10%_50V
- added D1, D2, D3: LESD5D5.0CT1G_C41399463, lcsc_footprints:C41399463_SOD-523_L1_2-W0_8-LS1_6-BI, symbol lcsc_imported:LESD5D5_0CT1G_C41399463
- added D4: 1N5819HW-7-F, lcsc_footprints:C82544_SOD-123_L2_7-W1_6-LS3_7-RD, symbol lcsc_imported:1N5819HW-7-F
- added U1: ESP32-S3-WROOM-1, RF_Module:ESP32-S3-WROOM-1, symbol RF_Module:ESP32-S3-WROOM-1
- added USB1: TYPE-C 16PIN 2MD(073), lcsc_footprints:C2765186_USB-C-SMD_TYPE-C-16PIN-2MD-073, symbol lcsc_imported:TYPE-C_16PIN_2MD(073)
Connections:
- new net: D3.2, D4.2 (A), USB1.A4B9 (VBUS), USB1.B4A9 (VBUS)
- new net: D1.2, USB1.A7 (Dn1), USB1.B7 (Dn2)
- new net: D2.2, USB1.A6 (Dp1), USB1.B6 (Dp2)
- new net EN: U1.3 (EN)
- new net ESP_3V3: C7.1, C8.1, U1.2 (3V3)
- new net GND: C11.2, C7.2, C8.2, D3.1, U1.1 (GND), U1.16 (IO46), U1.40 (GND), U1.41 (GND), USB1.13 (EH), USB1.14 (EH), USB1.A1B12 (GND), USB1.B1A12 (GND)
- new net IO0: U1.27 (IO0)
- new net USB_D+: D2.1, U1.13 (USB_D-)
- new net USB_D-: D1.1, U1.14 (USB_D+)
- new net VCC_5V: C11.1, D4.1 (K)
- no-connect marks 0 -> 2
Other:
- added sheet BOOT-RES (BOOT-RES.kicad_sch)
- added sheet POWER (POWER.kicad_sch)

Commit message: Battery charging IC
Parts:
- added CN1: S2B-PH-SM4-TB(LF)(SN), lcsc_footprints:C295747_CONN-SMD_P2_00_S2B-PH-SM4-TB-LF-SN, symbol lcsc_imported:S2B-PH-SM4-TB(LF)(SN)
Connections:
- net GND: now also CN1.2, CN1.3, CN1.4
- new net BAT: CN1.1
Other:
- added sheet BAT_CHRG (BAT_CHRG.kicad_sch)
- added sheet KeyBoard (Keyboard.kicad_sch)
- sheet POWER ports: added BAT_5V; removed VCC_5V
